File: arduino/arduino leds.kicad_pcb (KiCad board)
At the start: 2 copper layers, 99.1 x 49.5 mm, 23 parts, among them IC1 ATMEGA328-P

Commit message: Last changes
Parts:
- added C1: CAPAPOL, c_elec_4x5.8, F.Cu at (52.0, 38.0)
- added C2: C, C1, F.Cu at (84.0, 20.0)
- added P1: CONN_2, bornier2, F.Cu at (58.0, 23.0)
- added P2: CONN_2, bornier2, F.Cu at (91.0, 43.0)
- added P3: CONN_2, bornier2, F.Cu at (91.0, 30.0)
- added U1: 7805, TO220, F.Cu at (51.0, 29.0)
- moved R2 23.2 mm to (40.0, 51.0)
- moved R4 12.6 mm to (49.0, 44.0)
- moved R3 12.2 mm to (46.0, 48.0)
- turned D10 to 180 degrees
- turned D11 to 180 degrees
- turned D13 to 90 degrees
- turned D3 to 180 degrees
Connections:
- IC1 pad 22: (no net) -> GND
- IC1 pad 27: (no net) -> /BTN1
- IC1 pad 28: (no net) -> /BTN2
- IC1 pad 7: (no net) -> /VO
Routing:
- net /PIN6: track 73.9 -> 15.9 mm
- net /VO: track 0.00 -> 56.1 mm
- net N-0000036: track 65.2 -> 43.6 mm
- net /BTN1: track 0.00 -> 18.2 mm
- net N-0000037: track 134.3 -> 116.7 mm
- net /VI: track 0.00 -> 17.1 mm
- net N-0000010: track 31.7 -> 14.6 mm
- net /PIN5: track 20.1 -> 6.78 mm
- net /PIN7: track 19.0 -> 6.47 mm
- net /BTN2: track 0.00 -> 6.94 mm
- net N-0000017: track 35.2 -> 41.8 mm
- net /PIN11: track 18.7 -> 16.0 mm
- net N-000002: track 99.8 -> 101.6 mm
- net /PIN12: track 44.1 -> 43.0 mm
- net N-000005: track 7.30 -> 6.33 mm
Other:
- net class Default: trace_width 0.254 -> 0.654
- rule trace_min: 0.254 -> 0.654
